File: cm4-thinkpad.kicad_sch (KiCad schematic)
At the start: 15 parts

Commit message: finish charger circuit
Parts:
- added C? (x7): 0.1uF, symbol Device:C
- added C?: 220uF, symbol Device:C
- added C? (x2): 1uF, symbol Device:C
- added C?: 0.01uF, symbol Device:C
- added C? (x4): 10uF, symbol Device:C
- added C?: 2200pF, symbol Device:C
- added C?: 0.047uF, symbol Device:C
- added D?: D, symbol Device:D
- added L?: 4.7uH, symbol pspice:INDUCTOR
- added Q? (x2): SiS412DN, Package_SO:Vishay_PowerPAK_1212-8_Single, symbol CM4-Thinkpad:SiS412DN
- added Q?: FDS6680A, Package_SO:SOIC-8_3.9x4.9mm_P1.27mm, symbol CM4-Thinkpad:FDS6680A
- added R? (x3): 10k, Resistor_SMD:R_0603_1608Metric_Pad0.98x0.95mm_HandSolder, symbol Device:R
- added R? (x2): 10, symbol Device:R
- added R? (x2): 10m, symbol Device:R
- added R?: 100k, symbol Device:R
- added R? (x2): 4.02k, symbol Device:R
- added R?: 7.5, symbol Device:R
- added R?: 549k, symbol Device:R
- C?: symbol Device:CP -> Device:C
- Module? (x2): symbol CM4:ComputeModule4-CM4 -> CM4-Thinkpad:ComputeModule4-CM4
Connections:
- net EDP_EN is gone; now on net BQ_ACOK: Module?.24 (GPIO26)
- net +1.8v: no longer Module?.78 (GPIO_VREF(1.8v/3.3v_Input))
- net +3.3V: now also R?.1, R?.1, R?.1
- net +3.3v: now also Module?.78 (GPIO_VREF(1.8v/3.3v_Input)), R?.1
- net GND: now also U?.14 (GND), C?.1, C?.1, C?.1, C?.1, C?.1, C?.1, C?.2, C?.2, C?.2, C?.2, C?.2, Q?.1 (S), Q?.2 (S), Q?.3 (S), R?.2
- net I2C0_SCL: now also U?.8 (SDA), R?.2
- net I2C0_SDA: now also U?.9 (SCL), R?.2
- net at D?.1, Q?.5 (D), Q?.6 (D)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: now also C?.1, R?.1
- net VCC_SYS: now reaches U?.1 (ACN)
- net VCC_SYS: now also C?.1, C?.2, C?.2, C?.2, C?.2, Q?.5 (D), Q?.5 (D), Q?.6 (D), Q?.7 (D), Q?.8 (D), R?.2
- net BQ_ILIM: now reaches U?.10 (ILIM)
- net BQ_ILIM: now also R?.1, R?.2
- net at U?.11 (BATDRV): now also R?.1
- net at U?.12 (SRN): now also R?.1
- net at U?.13 (SRP): now also R?.1
- net at U?.15 (LODRV): now also Q?.4 (G)
- net at U?.16 (REGN): now also C?.1, D?.2 (A)
- net at U?.17 (BTST): now also C?.1, D?.1 (K)
- net at U?.18 (HIDRV): now also Q?.4 (G)
- net at U?.19 (PHASE): now also C?.2, L?.1, Q?.1 (S), Q?.2 (S), Q?.3 (S), Q?.5 (D)
- net at U?.2 (ACP): now also Q?.1 (S), Q?.2 (S), Q?.3 (S), C?.1, C?.1, C?.1, R?.1, R?.1
- net at U?.20 (VCC): now also C?.2, R?.2
- net at U?.3 (CMSRC): now also R?.2
- net BQ_ACOK: now reaches U?.5 (ACOK)
- net BQ_ACOK: now also R?.2
- net BQ_IOUT_ADC: now reaches U?.7 (IOUT)
- net BQ_IOUT_ADC: now also C?.1
- net at Q?.4 (G), R?.1: now also C?.2, C?.2
- net EDP_IRQ: no longer names the net of Module?.26 (GPIO19)
- new net: C?.1, L?.2, R?.1, R?.2
- new net: C?.2, Q?.4 (G), R?.2
- new net +VBAT: C?.1, C?.1, C?.2, C?.2, C?.2, Q?.1 (S), Q?.2 (S), Q?.3 (S), R?.2, R?.2
- no-connect marks 0 -> 2
Other:
- note added: "549k ~= 2.49A current limit optimal for a 65w charger"
- note added: "9v-20v"
- note added: "Charger Circuit"
- note added: "Indicators and pullups"
- note added: "RAC"
- note added: "make sure this does ADC probably not needed."
- note removed: "Indicators"
- moved on the sheet: D?, Q?, R?, U?
